File: hardware/enclosure/1v0_76x35_kpl/panel/Front_Panel_76x35/Front_Panel_76x35.kicad_pcb (KiCad board)
At the start: 2 copper layers, 76 x 35 mm, 11 parts

Commit message: Org June 2018
Other:
- board text added: "TXH"
- board text added: "TXL"
- board text added: "Tx1"
- board text removed: "TX1"
- board text removed: "TX2"
Changed lines of the file:
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@@
-(kicad_pcb (version 20170123) (host pcbnew "(2017-06-07 revision 51bed4bae)-makepkg")
+(kicad_pcb (version 4) (host pcbnew 4.0.7)
   (general
     (links 119)
     (no_connects 0)
-    (area 25.34 92.7 101.900001 128.200001)
+    (area 25.619999 92.929999 101.630001 127.950001)
     (thickness 1.6)
-    (drawings 276)
+    (drawings 265)
     (tracks 0)
     (zones 0)
@@
   (page A4)
   (layers
-    (0 F.Cu signal)
-    (31 B.Cu signal)
-    (32 B.Adhes user)
-    (33 F.Adhes user)
-    (34 B.Paste user)
-    (35 F.Paste user)
+    (0 F.Cu signal hide)
+    (31 B.Cu signal hide)
+    (32 B.Adhes user hide)
+    (33 F.Adhes user hide)
+    (34 B.Paste user hide)
+    (35 F.Paste user hide)
     (36 B.SilkS user)
     (37 F.SilkS user)
-    (38 B.Mask user)
-    (39 F.Mask user)
-    (40 Dwgs.User user)
-    (41 Cmts.User user)
-    (42 Eco1.User user)
-    (43 Eco2.User user)
+    (38 B.Mask user hide)
+    (39 F.Mask user hide)
+    (40 Dwgs.User user hide)
+    (41 Cmts.User user hide)
+    (42 Eco1.User user hide)
+    (43 Eco2.User user hide)
     (44 Edge.Cuts user)
     (45 Margin user hide)
@@
     (zone_45_only yes)
     (trace_min 0.2)
-    (segment_width 0.2)
+    (segment_width 0.5)
     (edge_width 0.02)
     (via_size 0.8)
@@
     (aux_axis_origin 25.6 92.9)
     (grid_origin 25.6 92.9)
-    (visible_elements 7FFFFFFF)
+    (visible_elements 7FFC3601)
     (pcbplotparams
       (layerselection 0x010f0_ffffffff)
@@
       (hpglpenspeed 20)
       (hpglpendiameter 15)
+      (hpglpenoverlay 2)
       (psnegative false)
       (psa4output false)
@@
   )
   (module Ohisja:SMA_test1 (layer B.Cu)
-    (at 90.05 113.73 180)
+    (at 77.05 99.73 180)
     (fp_text reference REF** (at 0 -7.7 180) (layer Dwgs.User)
       (effects (font (size 1 1) (thickness 0.15)))
@@
   )
   (module Ohisja:SMA_test1 (layer B.Cu)
-    (at 77.05 113.73 180)
+    (at 90.05 113.73 180)
     (fp_text reference REF** (at 0 -7.7 180) (layer Dwgs.User)
       (effects (font (size 1 1) (thickness 0.15)))
@@
   )
   (module Ohisja:SMA_test1 (layer B.Cu)
-    (at 90.05 99.73 180)
+    (at 77.05 113.73 180)
     (fp_text reference REF** (at 0 -7.7 180) (layer Dwgs.User)
       (effects (font (size 1 1) (thickness 0.15)))
@@
   )
   (module Ohisja:SMA_test1 (layer B.Cu)
-    (at 77.05 99.73 180)
+    (at 90.05 99.73 180)
     (fp_text reference REF** (at 0 -7.7 180) (layer Dwgs.User)
       (effects (font (size 1 1) (thickness 0.15)))
@@
       (xy 0.633926 0.143156) (xy 0.583106 0.213221) (xy 0.580402 0.21803) (xy 0.555092 0.274533)
       (xy 0.5756 0.288591) (xy 0.640127 0.276382)) (layer B.Mask) (width 0.01))
+  )
+  (gr_text Tx1 (at 77.1 121.4) (layer B.SilkS)
+    (effects (font (size 1.5 1.5) (thickness 0.3)) (justify mirror))
+  )
+  (gr_arc (start 80.2 96.1) (end 80.2 93.9) (angle 90) (layer B.SilkS) (width 0.5))
+  (gr_line (start 82.4 104) (end 82.4 110) (angle 90) (layer B.SilkS) (width 0.5))
+  (gr_arc (start 80.2 117.7) (end 82.4 117.5) (angle 90) (layer B.SilkS) (width 0.5))
+  (gr_arc (start 73.656034 117.84428) (end 71.606034 117.79428) (angle -91.39718103) (layer B.SilkS) (width 0.5))
+  (gr_line (start 73.7 119.9) (end 80.2 119.9) (angle 90) (layer B.SilkS) (width 0.5))
+  (gr_line (start 73.5 93.9) (end 80.2 93.9) (angle 90) (layer B.SilkS) (width 0.5))
+  (gr_arc (start 73.6 95.9) (end 71.6 96) (angle 90) (layer B.SilkS) (width 0.5))
+  (gr_line (start 71.6 117.8) (end 71.6 95.8) (angle 90) (layer B.SilkS) (width 0.5))
+  (gr_line (start 68.8 117.9) (end 68.8 110.03061) (layer B.SilkS) (width 0.5))
+  (gr_text tx1H (at 77.34 105.56) (layer F.SilkS)
+    (effects (font (size 1.6 1.6) (thickness 0.3)))
   )
   (gr_arc (start 27.63 125.94) (end 27.63 127.94) (angle 90) (layer Edge.Cuts) (width 0.02))
@@
   (gr_circle (center 29.58 96.93) (end 27.78 96.93) (layer B.Mask) (width 0.8))
   (gr_circle (center 97.575 96.925) (end 98.975 96.925) (layer Edge.Cuts) (width 0.02))
-  (gr_text L (at 90.05 106.03) (layer B.SilkS)
-    (effects (font (size 1.8 1.8) (thickness 0.3)) (justify mirror))
-  )
-  (gr_line (start 86.25 105.93) (end 80.95 105.93) (layer B.SilkS) (width 0.5))
-  (gr_text H (at 77.05 106.04489) (layer B.SilkS)
-    (effects (font (size 1.8 1.8) (thickness 0.3)) (justify mirror))
-  )
-  (gr_arc (start 73.34 103.86939) (end 71.29 103.81939) (angle -91.39718103) (layer B.SilkS) (width 0.5))
-  (gr_line (start 71.24 96.02) (end 71.29 103.81939) (layer B.SilkS) (width 0.5))
-  (gr_arc (start 73.29 95.98) (end 73.34 93.93) (angle -91.39718103) (layer B.SilkS) (width 0.5))
-  (gr_line (start 93.85 93.93) (end 73.35 93.93) (layer B.SilkS) (width 0.5))
-  (gr_arc (start 93.75 95.98061) (end 95.8 96.03061) (angle -91.39718103) (layer B.SilkS) (width 0.5))
-  (gr_line (start 95.8 103.9) (end 95.8 96.03061) (layer B.SilkS) (width 0.5))
-  (gr_arc (start 93.74939 103.9) (end 93.69939 105.95) (angle -91.39718103) (layer B.SilkS) (width 0.5))
-  (gr_text TX1 (at 97.85 103.63 90) (layer B.SilkS)
+  (gr_text "TXH\n" (at 97.85 103.63 90) (layer B.SilkS)
     (effects (font (size 2 2.2) (thickness 0.35)) (justify mirror))
   )
-  (gr_arc (start 73.29 109.98) (end 73.34 107.93) (angle -91.39718103) (layer B.SilkS) (width 0.5))
-  (gr_line (start 71.24 110.02) (end 71.29 117.81939) (layer B.SilkS) (width 0.5))
-  (gr_arc (start 73.34 117.86939) (end 71.29 117.81939) (angle -91.39718103) (layer B.SilkS) (width 0.5))
   (gr_arc (start 66.75 95.98061) (end 68.8 96.03061) (angle -91.39718103) (layer B.SilkS) (width 0.5))
   (gr_line (start 68.8 103.85) (end 68.8 96.03061) (layer B.SilkS) (width 0.5))
@@
     (effects (font (size 2 2.2) (thickness 0.35)) (justify mirror))
   )
-  (gr_text H (at 77.05 120.04489) (layer B.SilkS)
-    (effects (font (size 1.8 1.8) (thickness 0.3)) (justify mirror))
-  )
-  (gr_text L (at 90.05 120.03) (layer B.SilkS)
-    (effects (font (size 1.8 1.8) (thickness 0.3)) (justify mirror))
-  )
-  (gr_line (start 86.25 119.93) (end 80.95 119.93) (layer B.SilkS) (width 0.5))
-  (gr_line (start 93.85 107.93) (end 73.35 107.93) (layer B.SilkS) (width 0.5))
-  (gr_arc (start 93.75 109.98061) (end 95.8 110.03061) (angle -91.39718103) (layer B.SilkS) (width 0.5))
-  (gr_line (start 95.8 117.9) (end 95.8 110.03061) (layer B.SilkS) (width 0.5))
-  (gr_arc (start 93.74939 117.88) (end 93.69939 119.93) (angle -91.39718103) (layer B.SilkS) (width 0.5))
-  (gr_text TX2 (at 97.85 117.63 90) (layer B.SilkS)
+  (gr_text "TXL\n" (at 97.85 117.63 90) (layer B.SilkS)
     (effects (font (size 2 2.2) (thickness 0.35)) (justify mirror))
   )
@@
     (effects (font (size 2 2.2) (thickness 0.35)) (justify mirror))
   )
-  (gr_line (start 68.8 117.9) (end 68.8 110.03061) (layer B.SilkS) (width 0.5))
-  (gr_arc (start 66.74939 117.88) (end 66.69939 119.93) (angle -91.39718103) (layer B.SilkS) (width 0.5))
+  (gr_arc (start 66.74939 117.88) (end 66.69939 119.93) (angle -91.3) (layer B.SilkS) (width 0.5))
   (gr_arc (start 66.75 109.98061) (end 68.8 110.03061) (angle -91.39718103) (layer B.SilkS) (width 0.5))
   (gr_line (start 59.25 119.93) (end 53.95 119.93) (layer B.SilkS) (width 0.5))
@@
     (effects (font (size 1.6 1.6) (thickness 0.3)))
   )
-  (gr_text tx2H (at 77.31 107.95) (layer F.SilkS)
+  (gr_text tx1L (at 77.31 107.95) (layer F.SilkS)
     (effects (font (size 1.6 1.6) (thickness 0.3)))
   )
@@
     (effects (font (size 1.6 1.6) (thickness 0.3)))
   )
-  (gr_text tx1H (at 77.34 105.56) (layer F.SilkS)
+  (gr_text tx2H (at 90.37 105.56) (layer F.SilkS)
     (effects (font (size 1.6 1.6) (thickness 0.3)))
   )
-  (gr_text tx1L (at 90.37 105.56) (layer F.SilkS)
-    (effects (font (size 1.6 1.6) (thickness 0.3)))
-  )
